Commit message: added launch slam

File: urdf/multi_puzzlebot.urdf (robot description, URDF)
Before this commit: robot pname, 5 links, 4 joints
Links:
- added link laser_link
Joints:
- added joint laser_joint: type fixed, parent pname_base_link, child laser_link, origin xyz=0.0 0.0 0.15 rpy=0 0 0

File: urdf/puzzlebot.urdf (robot description, URDF)
Before this commit: robot puzzlebot, 5 links, 4 joints
Links:
- added link laser_link
Joints:
- added joint laser_joint: type fixed, parent base_link, child laser_link, origin xyz=0.0 0.0 0.1 rpy=0 0 0

Commit message: Kalman filter localization Done :D

File: urdf/multi_puzzlebot.urdf (robot description, URDF)
Before this commit: robot pname, 6 links, 5 joints
Links:
- added link camera_link
Joints:
- added joint camera_joint: type fixed, parent pname_base_link, child camera_link, origin xyz=0.1 0.0 0.0375 rpy=-1.57 0 -1.57

File: urdf/puzzlebot.urdf (robot description, URDF)
Before this commit: robot puzzlebot, 6 links, 5 joints
Links:
- added link camera_link
Joints:
- added joint camera_joint: type fixed, parent base_link, child camera_link, origin xyz=0.1 0.0 0.0375 rpy=-1.57 0 -1.57
